File: hardware/kicad/disctracker_sensor.kicad_sch (KiCad schematic)
At the start: 40 parts, among them J1 BAT+, J2 BAT-, M1 XIAO nRF52840 Sense, U1 LSM6DSV320X, U2 LSM6DSV320X, U3 LSM6DSV320X, U4 LSM6DSV320X, U5 LSM6DSV320X, U6 MMC5603NJ

Commit message: Add routed 4-layer PCB layout and JLCPCB fab files for the sensor board
56 mm round board, sensors on top (machine assembled), XIAO + battery + buzzer
on the bottom. In1 is a solid GND plane, In2 a +3V3 pour; Freerouting on the
signal layers, locked GND fan-out under each IMU, GND stitching vias. DRC is
clean with schematic parity (0 violations, 0 unconnected). XIAO VBAT/GND
underside pads become plated holes; its pad 18 is now left unconnected in the
schematic. Gerbers, drills, JLC BOM/CPL, STEP and renders in kicad/fab.

Co-Authored-By: Claude Opus 5.5 <noreply@anthropic.com>
Claude-Session: https://claude.ai/code/session_013WWMZni5TrjV9cuQFT1N1C
Parts:
- TP1: value trim +X -> trim NE
- TP2: value trim -X -> trim NW
- TP3: value trim +Y -> trim SW
- TP4: value trim -Y -> trim SE
Connections:
- net GND: no longer M1.18 (GND)
- no-connect marks 29 -> 30
Other:
- note added: "D0-D10 all used. D6 goes to JP1 (U5 chip-select or buzzer). VBUS, SWD, EN, NFC and underside GND pad 18 left unconnected (GND via pads 13 and 20; 19/20 are plated holes). Firmware: P1.11 (D6) high drive for the buzzer; charge current 100 mA (P0.13 low)."
- note added: "Trim pads at r = 22 mm on the diagonals (XIAO face); SW/SE sit opposite the buzzer. Holes locate the board on the pod's pins."
- note removed: "D0-D10 all used. D6 goes to JP1 (U5 chip-select or buzzer). VBUS, SWD, EN and NFC pads left unconnected. Firmware: P1.11 (D6) high drive for the buzzer; charge current 100 mA (P0.13 low)."
- note removed: "Trim pads: -Y pad sits opposite the buzzer; others for fine balance. Holes locate the board on the pod's pins."
Changed lines of the file:
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@@
   (no_connect (at 52.07 34.29))
   (no_connect (at 55.88 34.29))
-  (wire (pts (xy 59.69 34.29) (xy 59.69 31.75)) (stroke (width 0) (type default)))
-  (label "GND" (at 59.69 31.75 90) (fields_autoplaced yes) (effects (font (size 1.27 1.27)) (justify left bottom)))
+  (no_connect (at 59.69 34.29))
   (wire (pts (xy 48.26 71.12) (xy 48.26 73.66)) (stroke (width 0) (type default)))
   (label "VBAT" (at 48.26 73.66 270) (fields_autoplaced yes) (effects (font (size 1.27 1.27)) (justify right bottom)))
@@
   (wire (pts (xy 99.06 92.71) (xy 99.06 95.25)) (stroke (width 0) (type default)))
   (label "GND" (at 99.06 95.25 270) (fields_autoplaced yes) (effects (font (size 1.27 1.27)) (justify right bottom)))
-  (text "D0-D10 all used. D6 goes to JP1 (U5 chip-select or buzzer).\nVBUS, SWD, EN and NFC pads left unconnected.\nFirmware: P1.11 (D6) high drive for the buzzer;\ncharge current 100 mA (P0.13 low)." (exclude_from_sim no) (at 15.24 92.71 0) (effects (font (size 1.27 1.27)) (justify left top)))
+  (text "D0-D10 all used. D6 goes to JP1 (U5 chip-select or buzzer).\nVBUS, SWD, EN, NFC and underside GND pad 18 left unconnected\n(GND via pads 13 and 20; 19/20 are plated holes).\nFirmware: P1.11 (D6) high drive for the buzzer;\ncharge current 100 mA (P0.13 low)." (exclude_from_sim no) (at 15.24 92.71 0) (effects (font (size 1.27 1.27)) (justify left top)))
   (rectangle (start 114.3 20.32) (end 406.4 160.02) (stroke (width 0.15) (type dash)) (fill (type none)))
   (text "Motion sensors · 5x LSM6DSV320X on shared SPI (sensor face, all same orientation)" (exclude_from_sim no) (at 115.57 21.59 0) (effects (font (size 2 2) (bold yes)) (justify left top)))
@@
   (symbol (lib_id "Connector:TestPoint") (at 330.2 190.5 0) (unit 1) (exclude_from_sim no) (in_bom no) (on_board yes) (dnp no)
   (property "Reference" "TP1" (at 332.74 184.15 0) (effects (font (size 1.27 1.27)) (justify left)))
-  (property "Value" "trim +X" (at 332.74 186.055 0) (effects (font (size 1.27 1.27)) (justify left)))
+  (property "Value" "trim NE" (at 332.74 186.055 0) (effects (font (size 1.27 1.27)) (justify left)))
   (property "Footprint" "TestPoint:TestPoint_Pad_3.0x3.0mm" (at 330.2 190.5 0) (effects (font (size 1.27 1.27)) (hide yes)))
   (property "Datasheet" "" (at 330.2 190.5 0) (effects (font (size 1.27 1.27)) (hide yes)))
@@
   (symbol (lib_id "Connector:TestPoint") (at 347.98 190.5 0) (unit 1) (exclude_from_sim no) (in_bom no) (on_board yes) (dnp no)
   (property "Reference" "TP2" (at 350.52 184.15 0) (effects (font (size 1.27 1.27)) (justify left)))
-  (property "Value" "trim -X" (at 350.52 186.055 0) (effects (font (size 1.27 1.27)) (justify left)))
+  (property "Value" "trim NW" (at 350.52 186.055 0) (effects (font (size 1.27 1.27)) (justify left)))
   (property "Footprint" "TestPoint:TestPoint_Pad_3.0x3.0mm" (at 347.98 190.5 0) (effects (font (size 1.27 1.27)) (hide yes)))
   (property "Datasheet" "" (at 347.98 190.5 0) (effects (font (size 1.27 1.27)) (hide yes)))
@@
   (symbol (lib_id "Connector:TestPoint") (at 365.76 190.5 0) (unit 1) (exclude_from_sim no) (in_bom no) (on_board yes) (dnp no)
   (property "Reference" "TP3" (at 368.3 184.15 0) (effects (font (size 1.27 1.27)) (justify left)))
-  (property "Value" "trim +Y" (at 368.3 186.055 0) (effects (font (size 1.27 1.27)) (justify left)))
+  (property "Value" "trim SW" (at 368.3 186.055 0) (effects (font (size 1.27 1.27)) (justify left)))
   (property "Footprint" "TestPoint:TestPoint_Pad_3.0x3.0mm" (at 365.76 190.5 0) (effects (font (size 1.27 1.27)) (hide yes)))
   (property "Datasheet" "" (at 365.76 190.5 0) (effects (font (size 1.27 1.27)) (hide yes)))
@@
   (symbol (lib_id "Connector:TestPoint") (at 383.54 190.5 0) (unit 1) (exclude_from_sim no) (in_bom no) (on_board yes) (dnp no)
   (property "Reference" "TP4" (at 386.08 184.15 0) (effects (font (size 1.27 1.27)) (justify left)))
-  (property "Value" "trim -Y" (at 386.08 186.055 0) (effects (font (size 1.27 1.27)) (justify left)))
+  (property "Value" "trim SE" (at 386.08 186.055 0) (effects (font (size 1.27 1.27)) (justify left)))
   (property "Footprint" "TestPoint:TestPoint_Pad_3.0x3.0mm" (at 383.54 190.5 0) (effects (font (size 1.27 1.27)) (hide yes)))
   (property "Datasheet" "" (at 383.54 190.5 0) (effects (font (size 1.27 1.27)) (hide yes)))
@@
   (property "Description" "Pod alignment pin hole, r = 25.6 mm at 30 / 150 / 250 deg" (at 381 210.82 0) (effects (font (size 1.27 1.27)) (hide yes)))
   (instances (project "disctracker_sensor" (path "/ed8d3162-2461-588e-942b-e23f59aa8ac7" (reference "H3") (unit 1)))))
-  (text "Trim pads: -Y pad sits opposite the buzzer; others for fine balance.\nHoles locate the board on the pod's pins." (exclude_from_sim no) (at 320.04 222.25 0) (effects (font (size 1.27 1.27)) (justify left top)))
+  (text "Trim pads at r = 22 mm on the diagonals (XIAO face); SW/SE sit opposite the buzzer.\nHoles locate the board on the pod's pins." (exclude_from_sim no) (at 320.04 222.25 0) (effects (font (size 1.27 1.27)) (justify left top)))
   (rectangle (start 12.7 243.84) (end 226.06 284.48) (stroke (width 0.15) (type dash)) (fill (type none)))
   (text "Board notes" (exclude_from_sim no) (at 13.97 245.11 0) (effects (font (size 2 2) (bold yes)) (justify left top)))
